Commit message: some updates

File: urdf/scara-robot.urdf (robot description, URDF)
Before this commit: robot scara, 7 links, 6 joints
Links:
- added link world
- link base_link: mass None -> 10; geometry collision cylinder length=1.2 radius=0.15; visual cylinder length=1.2 radius=0.15
- link first_joint: mass None -> 0; geometry collision cylinder length=0.3 radius=0.15; visual cylinder length=0.3 radius=0.15
- link first_link: mass None -> 0; geometry collision box size=0.9 0.15 0.3; visual box size=0.9 0.15 0.3
- link second_joint: mass None -> 0; geometry collision cylinder length=0.3 radius=0.15; visual cylinder length=0.3 radius=0.15
- link second_link: mass None -> 0; geometry collision box size=0.9 0.15 0.3; visual box size=0.9 0.15 0.3
- link third_link: mass None -> 0; geometry collision cylinder length=0.6 radius=0.05; visual cylinder length=0.6 radius=0.05
- link wrist_link: mass None -> 0; geometry collision box size=0.01 0.05 0.1; visual box size=0.01 0.05 0.1
Joints:
- added joint fixed: type fixed, parent world, child base_link, origin xyz=0 0 0

Commit message: fixed model

File: urdf/scara-robot.urdf (robot description, URDF)
Before this commit: robot scara, 8 links, 7 joints
Links:
- removed link first_joint
- removed link second_joint
- removed link wrist_link
- added link cover1_left; visual cylinder length=0.1 radius=0.1
- added link cover1_right; visual cylinder length=0.1 radius=0.1
- added link cover2_left; visual cylinder length=0.1 radius=0.1
- added link cover2_right; visual cylinder length=0.1 radius=0.1
- link base_link: mass 10 -> 1; geometry collision cylinder length=0.5 radius=0.1; visual cylinder length=0.5 radius=0.1
- link first_link: mass 0 -> 1; geometry collision box size=0.9 0.15 0.1; visual box size=0.9 0.15 0.1
- link second_link: mass 0 -> 1; geometry collision box size=0.9 0.15 0.1; visual box size=0.9 0.15 0.1
- link third_link: mass 0 -> 1
Joints:
- removed joint base_to_first_link
- removed joint first_joint_to_second_link
- removed joint first_link_to_first_joint
- removed joint second_joint_to_third_joint
- removed joint second_link_to_second_joint
- removed joint third_link_to_wrist_link
- added joint base_to_first_joint: type revolute, parent base_link, child first_link, origin xyz=0 0 0.5 rpy=0 0 0, axis 0 0 1, limit lower=-2.6 upper=2.6 effort=1000.0 velocity=0.5
- added joint first_to_second_joint: type revolute, parent first_link, child second_link, origin xyz=0.9 0 0.1 rpy=0 0 0, axis 0 0 1, limit lower=-2.6 upper=2.6 effort=1000.0 velocity=0.5
- added joint left_cover_link1: type fixed, parent first_link, child cover1_left
- added joint left_cover_link2: type fixed, parent second_link, child cover2_left
- added joint right_cover_link1: type fixed, parent first_link, child cover1_right
- added joint right_cover_link2: type fixed, parent second_link, child cover2_right
- added joint second_to_third_joint: type prismatic, parent second_link, child third_link, origin xyz=0.9 0 0 rpy=0 0 0, axis 0 0 1, limit lower=-0.30 upper=0.30 effort=1000.0 velocity=0.5
- joint fixed: origin xyz=0 0 0 -> (none)

Commit message: added moving in XY

File: urdf/scara-robot.urdf (robot description, URDF)
Before this commit: robot SCARA, 9 links, 8 joints
Links:
- link base_link: mass 1 -> 0.1
- link first_link: mass 1 -> 0.1
- link second_link: mass 1 -> 0.1
- link third_link: mass 1 -> 0.1
Joints:
- joint base_to_first_joint: limit lower=-2.6 upper=2.6 effort=1000.0 velocity=0.5 -> lower=-2.6 effort=1000.0 velocity=0.1
- joint first_to_second_joint: limit lower=-2.6 upper=2.6 effort=1000.0 velocity=0.5 -> lower=-2.6 upper=2.6 effort=1000.0 velocity=0.1
- joint second_to_third_joint: limit lower=-0.30 upper=0.30 effort=1000.0 velocity=0.5 -> lower=-0.30 upper=0.30 effort=1000.0 velocity=0.1

Commit message: bug fixed

File: urdf/scara-robot.urdf (robot description, URDF)
Before this commit: robot SCARA, 9 links, 8 joints
Joints:
- joint base_to_first_joint: limit lower=-2.6 effort=1000.0 velocity=0.1 -> lower=-2.6 upper=2.6 effort=1000.0 velocity=0.1
